File: womierk66-pcb/womierk66-pcb.sch (KiCad schematic (older format))
At the start: 12 parts, among them U1 ATmega32U4-AU

Commit message: Part 4 done, part 5 now.
Parts:
- added F?: 500mA, symbol Device:Polyfuse_Small
- added USB?: Molex-0548190589, symbol random-keyboard-parts:Molex-0548190589
Connections:
- net labels added: VCC
- wire segments 41 -> 48
Changed lines of the file:
@@
 Wire Wire Line
 	3350 1650 3350 1450
+$Comp
+L random-keyboard-parts:Molex-0548190589 USB?
+U 1 1 6100CBE2
+P 6500 2250
+F 0 "USB?" V 7037 2217 60  0000 C CNN
+F 1 "Molex-0548190589" V 6931 2217 60  0000 C CNN
+F 2 "" H 6500 2250 60  0001 C CNN
+F 3 "" H 6500 2250 60  0001 C CNN
+	1    6500 2250
+	0    -1   -1   0
+$EndComp
+$Comp
+L Device:Polyfuse_Small F?
+U 1 1 61010CDC
+P 7350 2050
+F 0 "F?" V 7145 2050 50  0000 C CNN
+F 1 "500mA" V 7236 2050 50  0000 C CNN
+F 2 "" H 7400 1850 50  0001 L CNN
+F 3 "~" H 7350 2050 50  0001 C CNN
+	1    7350 2050
+	0    1    1    0
+$EndComp
+$Comp
+L power:+5V #PWR?
+U 1 1 61012634
+P 7800 2050
+F 0 "#PWR?" H 7800 1900 50  0001 C CNN
+F 1 "+5V" H 7815 2223 50  0000 C CNN
+F 2 "" H 7800 2050 50  0001 C CNN
+F 3 "" H 7800 2050 50  0001 C CNN
+	1    7800 2050
+	1    0    0    -1
+$EndComp
+$Comp
+L power:VCC #PWR?
+U 1 1 61013A62
+P 7000 2050
+F 0 "#PWR?" H 7000 1900 50  0001 C CNN
+F 1 "VCC" H 7017 2223 50  0000 C CNN
+F 2 "" H 7000 2050 50  0001 C CNN
+F 3 "" H 7000 2050 50  0001 C CNN
+	1    7000 2050
+	1    0    0    -1
+$EndComp
+Wire Wire Line
+	6800 2050 7000 2050
+Connection ~ 7000 2050
+Wire Wire Line
+	7000 2050 7250 2050
+Wire Wire Line
+	7450 2050 7800 2050
+Text GLabel 7150 2250 2    50   Input ~ 0
+D+
+Text GLabel 7150 2150 2    50   Input ~ 0
+D-
+Wire Wire Line
+	7150 2150 6800 2150
+Wire Wire Line
+	6800 2250 7150 2250
+$Comp
+L power:GND #PWR?
+U 1 1 61017E19
+P 7150 2500
+F 0 "#PWR?" H 7150 2250 50  0001 C CNN
+F 1 "GND" H 7155 2327 50  0000 C CNN
+F 2 "" H 7150 2500 50  0001 C CNN
+F 3 "" H 7150 2500 50  0001 C CNN
+	1    7150 2500
+	1    0    0    -1
+$EndComp
+Wire Wire Line
+	6800 2450 7150 2450
+Wire Wire Line
+	7150 2450 7150 2500
 $EndSCHEMATC
